File: updated-withrelay/updated-withrelay/pressure-elec-board.kicad_sch (KiCad schematic)
At the start: 40 parts, among them IC1 DAC82001DRXR, J1 Screw_Terminal_01x03, J2 Screw_Terminal_01x03, J3 Screw_Terminal_01x03, J4 Screw_Terminal_01x03, J5 Screw_Terminal_01x03, K2 ALQ305, Q1 IRF540N, Q2 BSS138, Q3 BSS138, SW1 SW_DPST, U1 mpx2200, U2 ITV1031_smc, U4 MCP3301, U5 INA125P, U6 MCP3301, U7 PicoW

Commit message: Modified pcb to include two pressure rigs
Parts:
- added C3, C4: .1 uF, PCM_Capacitor_SMD_AKL:C_1206_3216Metric_Pad1.42x1.75mm, symbol PCM_Generic:C,IEC
- added IC2: DAC82001DRXR, DAC:SON50P250X250X80-10N, symbol DAC82001DRXR:DAC82001DRXR
- added J6: Screw_Terminal_01x03, TerminalBlock:TerminalBlock_Altech_AK300-2_P5.00mm, symbol Connector:Screw_Terminal_01x02
- added J7: Screw_Terminal_01x03, TerminalBlock:TerminalBlock_Altech_AK300-3_P5.00mm, symbol Connector:Screw_Terminal_01x03
- added Q4, Q5: BSS138, Package_TO_SOT_SMD_AKL:SOT-23, symbol PCM_Transistor_MOSFET_AKL:BSS138
- added R14, R4: 10 k, Resistor_SMD:R_0402_1005Metric, symbol PCM_Generic-50:R,IEC
- added R15: 5 k, Resistor_SMD:R_0402_1005Metric, symbol PCM_Generic-50:R,IEC
- added R16, R17, R18, R19: 10k, Resistor_THT:R_Axial_DIN0204_L3.6mm_D1.6mm_P7.62mm_Horizontal, symbol Device:R
- added R20: 810, Resistor_THT:R_Axial_DIN0204_L3.6mm_D1.6mm_P7.62mm_Horizontal, symbol Device:R
- added U10: mpx2200, MPX:MPX2200, symbol Sensor_Pressure:mpx2200
- added U11: INA125P, INA125P:ina125p_bigger_pads, symbol INA125P:INA125P
- added U12, U8: MCP3301, ADC:Microchip-MCP3301-CI_P-Manufacturer_Recommended, symbol Analog_ADC:MCP3301
- added U3: ITV1031_smc, symbol pressure_regulator:ITV1031_smc
Connections:
- net +12V: now also K2.NO, U3.1 (V_supply); no longer K2.C1, K2.COM
- net 3.3V: now also C4.2 (-), IC2.10 (VREF)
- net 5V: now also D1.2 (A), J4.1 (Pin_1), K2.C1, C3.2 (-), IC2.1 (VDD), R15.1 (+), U10.3 (V_supply), U11.1 (V+), U11.2 (~{SLEEP}), U12.1 (Vref), U12.8 (Vdd), U8.1 (Vref), U8.8 (Vdd)
- net ADC_1_ACTIVE: now also U7.15 (GPIO11), U12.5 (~{CS}/SHDN); no longer U7.10 (GPIO7)
- net ADC_2_ACTIVE: now also U7.14 (GPIO10), U8.5 (~{CS}/SHDN); no longer U7.9 (GPIO6)
- net CLK: now also U7.9 (GPIO6), IC2.6 (SCLK), U12.7 (CLK), U8.7 (CLK)
- net DAC_ACTIVE: now also U7.16 (GPIO12), IC2.7 (~{SYNC}), R15.2 (-); no longer U7.11 (GPIO8)
- net GND: now also C1.1 (+), C2.1 (+), K2.C2, Q1.3 (S), C3.1 (+), C4.1 (+), IC2.4 (AGND), J6.2 (Pin_2), R14.1 (+), R4.1 (+), U10.1 (GND), U11.12 (VREFCOM), U11.3 (V-), U11.5 (IAREF), U12.3 (IN-), U12.4 (Vss), U3.2 (GND), U8.3 (IN-), U8.4 (Vss)
- net GNDPWR: now also K2.COM; no longer K2.NO
- net GPIO5: now also U7.29 (GPIO22); no longer U7.7 (GPIO5)
- net HV_REF: now also R17.1, R19.1
- net LV_REF: now also Q4.1 (G), Q5.1 (G), R16.1, R18.1
- net MISO renamed MISO_reg1
- net MISO_reg1: now also U8.6 (Dout); no longer U4.6 (Dout)
- net MISO_3V renamed MISO_3V_reg1
- net MOSI renamed MOSI_reg2
- net MOSI_reg2: now also U7.10 (GPIO7); no longer U7.5 (GPIO3)
- net MOSI_5V renamed MOSI_5V_reg2
- net pressure_input renamed pressure_input1
- net pressure_input1: now also IC2.2 (VOUT); no longer IC1.2 (VOUT)
- net pressure_output renamed pressure_output1
- net pressure_output1: no longer U4.2 (IN+)
- new net: U11.10 (VO), U11.11 (SENSE), U12.2 (IN+)
- new net: U10.2 (+out), U11.6 (V+IN)
- new net: U10.4 (-out), U11.7 (V-IN)
- new net: R20.1, U11.8 (RG)
- new net: R20.2, U11.9 (RG)
- new net: IC2.3 (RSTSEL), R4.2 (-)
- new net: IC2.5 (~{RESET}), R14.2 (-)
- new net MISO_3V_reg2: Q5.2 (S), R18.2, U7.11 (GPIO8)
- new net MISO_reg2: Q5.3 (D), R19.2, U12.6 (Dout), U4.6 (Dout)
- new net MOSI_5V_reg1: IC2.8 (SDIN), Q4.3 (D), R17.2
- new net MOSI_reg1: Q4.2 (S), R16.2, U7.5 (GPIO3)
- new net pressure_input2: IC1.2 (VOUT), J6.1 (Pin_1), J7.1 (Pin_1), U3.3 (input_signal)
- new net pressure_output2: J7.2 (Pin_2), U3.4 (output_signals)
- new net pressure_output_reg1: U8.2 (IN+)
- new net pressure_output_reg2: U4.2 (IN+)
Other:
- note added: "adjust this"
- note added: "drain"
- note added: "gate"
- note added: "source"
- moved on the sheet: C1, C1-?, C2, C?, D1, IC1, J1, J2, J3, J4, J5, K2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
